Commit message: Added actual models and fully defined joint movement

File: urdf/thor.urdf.xacro (robot description, xacro)
@@ -1,8 +1,9 @@
 <?xml version="1.0"?>
-<robot name="thor">
+<robot xmlns:xacro="http://ros.org/wiki/xacro" name="thor">
+  <property name="M_PI" value="3.1415926535897931" />
   <link name="thor_base_link">
     <visual>
       <geometry>
-        <mesh scale="0.001 0.001 0.001" filename="package://thor_description/meshes/BaseBot.stl"/>
+        <mesh filename="package://thor_description/meshes/thor_base_link.stl"/>
       </geometry>
       <origin xyz="0 0 0" rpy="0 0 0"/>
@@ -15,5 +16,5 @@
     <visual>
       <geometry>
-        <mesh scale="0.001 0.001 0.001" filename="package://thor_description/meshes/Art1Body.stl"/>
+        <mesh filename="package://thor_description/meshes/thor_art1_link.stl"/>
       </geometry>
       <origin xyz="0 0 0" rpy="0 0 0"/>
@@ -26,7 +27,7 @@
     <visual>
       <geometry>
-        <box size="0.3 0.15 0.5"/>
+        <mesh filename="package://thor_description/meshes/thor_art2_link.stl"/>
       </geometry>
-      <origin xyz="0 0 0" rpy="0 0 0"/>
+      <origin xyz="0 .055 0" rpy="0 0 0"/>
       <material name="green">
         <color rgba="0 1 0 1"/>
@@ -36,11 +37,11 @@
   <link name="thor_art3_link" >
     <visual>
-      <geometry>
-        <cylinder length="0.2" radius="0.15"/>
-      </geometry>
-      <origin xyz="0 0 0" rpy="0 0 0"/>
-      <material name="yellow">
+    	<geometry>
+      	  <mesh filename="package://thor_description/meshes/thor_art3_link.stl"/>
+	</geometry>
+      	<origin xyz="0 -.0375 0" rpy="0 0 0"/>
+      	<material name="yellow">
         <color rgba="1 1 0 1"/>
-      </material>
+        </material>
     </visual>
   </link>
@@ -48,7 +49,7 @@
     <visual>
       <geometry>
-        <cylinder length="0.2" radius="0.15"/>
+	<mesh filename="package://thor_description/meshes/thor_art4_link.stl"/>
       </geometry>
-      <origin xyz="0 0 0" rpy="0 0 0"/>
+      <origin xyz="0 -.0025 0" rpy="0 0 0"/>
       <material name="red">
         <color rgba="1 0 0 1"/>
@@ -59,5 +60,5 @@
     <visual>
       <geometry>
-        <cylinder length="0.2" radius="0.15"/>
+	<mesh filename="package://thor_description/meshes/thor_art5_link.stl"/>
       </geometry>
       <origin xyz="0 0 0" rpy="0 0 0"/>
@@ -70,5 +71,5 @@
     <visual>
       <geometry>
-        <cylinder length="0.2" radius="0.15"/>
+        <mesh filename="package://thor_description/meshes/thor_art6_link.stl"/>
       </geometry>
       <origin xyz="0 0 0" rpy="0 0 0"/>
@@ -81,42 +82,42 @@
     <parent link="thor_base_link"/>
     <child link="thor_art1_link"/>
-    <origin xyz="0 0 .104" rpy="0 0 0" />
+    <origin xyz="0 0 .105" rpy="0 0 0" />
     <axis xyz="0 0 1" />
-    <limit effort="1000.0" lower="0.0" upper="6.283" velocity="0.5"/>
+    <limit effort="1.0" lower="-${M_PI}" upper="${M_PI}" velocity="0.5"/>
   </joint>
   <joint name="thor_art2_joint" type="revolute">
     <parent link="thor_art1_link"/>
     <child link="thor_art2_link"/>
-    <origin xyz="0 0 .195" rpy="0 0 0" />
-    <axis xyz="1 0 0" />
-    <limit effort="1000.0" lower="0.0" upper="3.142" velocity="0.5"/>
+    <origin xyz="0 0 .100" rpy="0 0 0" />
+    <axis xyz="0 1 0" />
+    <limit effort="1.0" lower="-${M_PI/2}" upper="${M_PI/2}" velocity="0.5"/>
   </joint>
   <joint name="thor_art3_joint" type="revolute">
     <parent link="thor_art2_link"/>
     <child link="thor_art3_link"/>
-    <origin xyz="0 0 .3392" rpy="0 0 0" />
-    <axis xyz="1 0 0" />
-    <limit effort="1000.0" lower="0.0" upper="6.283" velocity="0.5"/>
+    <origin xyz="0 0 .160" rpy="0 0 0" />
+    <axis xyz="0 1 0" />
+    <limit effort="1.0" lower="-${M_PI}" upper="${M_PI}" velocity="0.5"/>
   </joint>
   <joint name="thor_art4_joint" type="revolute">
     <parent link="thor_art3_link"/>
     <child link="thor_art4_link"/>
-    <origin xyz="0 0 .4263" rpy="0 0 0" />
+    <origin xyz="0 0 .090" rpy="0 0 0" />
     <axis xyz="0 0 1" />
-    <limit effort="1000.0" lower="0.0" upper="6.283" velocity="0.5"/>
+    <limit effort="1.0" lower="-${M_PI}" upper="${M_PI}" velocity="0.5"/>
   </joint>
   <joint name="thor_art5_joint" type="revolute">
     <parent link="thor_art4_link"/>
     <child link="thor_art5_link"/>
-    <origin xyz="0 0 0.52955" rpy="0 0 0" />
-    <axis xyz="1 0 0" />
-    <limit effort="1000.0" lower="0.0" upper="3.142" velocity="0.5"/>
+    <origin xyz="0 0 0.100" rpy="0 0 0" />
+    <axis xyz="0 1 0" />
+    <limit effort="1.0" lower="-${M_PI/2}" upper="${M_PI/2}" velocity="0.5"/>
   </joint>
   <joint name="thor_art6_joint" type="revolute">
     <parent link="thor_art5_link"/>
     <child link="thor_art6_link"/>
-    <origin xyz="0 0 0.52955" rpy="0 0 0" />
+    <origin xyz="0 0 .070" rpy="0 0 0" />
     <axis xyz="0 0 1" />
-    <limit effort="1000.0" lower="0.0" upper="6.283" velocity="0.5"/>
+    <limit effort="1000.0" lower="-${M_PI}" upper="${M_PI}" velocity="0.5"/>
   </joint>
 </robot>
